Commit message: Added arm_gripper move_group and rviz config

File: ur_moveit_config/srdf/ur_macro.srdf.xacro (robot description, xacro)
@@ -13,4 +13,9 @@
     <group name="${prefix}${name}_manipulator">
       <chain base_link="${prefix}base_link" tip_link="${prefix}tool0" />
+    </group>
+    <group name="${prefix}arm_gripper">
+        <group name="${prefix}${name}_manipulator" />
+        <joint name="${prefix}gripper_grasp_point_joint"/>
+        <link name="${prefix}gripper_grasp_point"/>
     </group>
     <!--GROUP STATES - Purpose - Define a named state for a particular group, in terms of joint values. This is useful to define states like 'folded arms'-->
@@ -39,4 +44,44 @@
       <joint name="${prefix}wrist_3_joint" value="-0.11" />
     </group_state>
+    <group_state name="${prefix}test_configuration" group="${prefix}arm_gripper">
+      <joint name="${prefix}elbow_joint" value="1.4" />
+      <joint name="${prefix}shoulder_lift_joint" value="-1.62" />
+      <joint name="${prefix}shoulder_pan_joint" value="1.54" />
+      <joint name="${prefix}wrist_1_joint" value="-1.2" />
+      <joint name="${prefix}wrist_2_joint" value="-1.6" />
+      <joint name="${prefix}wrist_3_joint" value="-0.0" />
+    </group_state>
+    <group_state name="${prefix}pre_picking" group="${prefix}arm_gripper">
+      <joint name="${prefix}elbow_joint" value="1.4" />
+      <joint name="${prefix}shoulder_lift_joint" value="-1.62" />
+      <joint name="${prefix}shoulder_pan_joint" value="1.54" />
+      <joint name="${prefix}wrist_1_joint" value="-1.35" />
+      <joint name="${prefix}wrist_2_joint" value="-1.6" />
+      <joint name="${prefix}wrist_3_joint" value="-0.0" />
+    </group_state>
+    <group_state name="${prefix}picking" group="${prefix}arm_gripper">
+      <joint name="${prefix}elbow_joint" value="1.605" />
+      <joint name="${prefix}shoulder_lift_joint" value="-1.64" />
+      <joint name="${prefix}shoulder_pan_joint" value="1.54" />
+      <joint name="${prefix}wrist_1_joint" value="-1.57" />
+      <joint name="${prefix}wrist_2_joint" value="-1.605" />
+      <joint name="${prefix}wrist_3_joint" value="-0.0" />
+    </group_state>
+    <group_state name="${prefix}pre_drop" group="${prefix}arm_gripper">
+      <joint name="${prefix}elbow_joint" value="1.37" />
+      <joint name="${prefix}shoulder_lift_joint" value="-1.59" />
+      <joint name="${prefix}shoulder_pan_joint" value="1.81" />
+      <joint name="${prefix}wrist_1_joint" value="-1.36" />
+      <joint name="${prefix}wrist_2_joint" value="-1.61" />
+      <joint name="${prefix}wrist_3_joint" value="0.26" />
+    </group_state>
+    <group_state name="${prefix}drop_off" group="${prefix}arm_gripper">
+      <joint name="${prefix}elbow_joint" value="1.57" />
+      <joint name="${prefix}shoulder_lift_joint" value="-1.61" />
+      <joint name="${prefix}shoulder_pan_joint" value="1.80" />
+      <joint name="${prefix}wrist_1_joint" value="-1.54" />
+      <joint name="${prefix}wrist_2_joint" value="-1.61" />
+      <joint name="${prefix}wrist_3_joint" value="0.26" />
+    </group_state>
     <!--END EFFECTOR - Purpose - Represent information about an end effector.-->
     <!--VIRTUAL JOINT - Purpose - this element defines a virtual joint between a robot link and an external frame of reference (considered fixed with respect to the robot)-->

Commit message: added gripper to the srdf

File: ur_moveit_config/srdf/ur_macro.srdf.xacro (robot description, xacro)
@@ -14,4 +14,7 @@
       <chain base_link="${prefix}base_link" tip_link="${prefix}tool0" />
     </group>
+    <group name="${prefix}gripper">
+      <chain base_link="${prefix}robotiq_85_base_link" tip_link="${prefix}robotiq_85_left_knuckle_link" />
+    </group>
     <group name="${prefix}arm_gripper">
         <group name="${prefix}${name}_manipulator" />
@@ -20,4 +23,10 @@
     </group>
     <!--GROUP STATES - Purpose - Define a named state for a particular group, in terms of joint values. This is useful to define states like 'folded arms'-->
+     <group_state name="${prefix}open" group="${prefix}gripper">
+      <joint name="${prefix}robotiq_85_left_knuckle_joint" value="0.0" />
+    </group_state>
+    <group_state name="${prefix}close" group="${prefix}gripper">
+      <joint name="${prefix}robotiq_85_left_knuckle_joint" value="8.0" />
+    </group_state>
     <group_state name="${prefix}home" group="${prefix}${name}_manipulator">
       <joint name="${prefix}elbow_joint" value="0" />

Commit message: adjusted srdf

File: ur_moveit_config/srdf/ur_macro.srdf.xacro (robot description, xacro)
@@ -16,4 +16,9 @@
     <group name="${prefix}gripper">
       <chain base_link="${prefix}robotiq_85_base_link" tip_link="${prefix}robotiq_85_left_knuckle_link" />
+      <link name="${prefix}robotiq_85_base_link"/>
+      <link name="${prefix}robotiq_85_left_knuckle_link"/>
+      <link name="${prefix}robotiq_85_right_knuckle_link"/>
+      <joint name="${prefix}robotiq_85_left_knuckle_joint"/>
+      <joint name="${prefix}robotiq_85_right_knuckle_joint"/>
     </group>
     <group name="${prefix}arm_gripper">
@@ -27,5 +32,5 @@
     </group_state>
     <group_state name="${prefix}close" group="${prefix}gripper">
-      <joint name="${prefix}robotiq_85_left_knuckle_joint" value="8.0" />
+      <joint name="${prefix}robotiq_85_left_knuckle_joint" value="0.8" />
     </group_state>
     <group_state name="${prefix}home" group="${prefix}${name}_manipulator">
