Commit message: fused ur and robotiq_gripper

File: ur_moveit_config/srdf/ur.srdf.xacro (robot description, xacro)
@@ -4,6 +4,9 @@
   <xacro:arg name="name" default="ur"/>
   <!-- parameters -->
-  <xacro:arg name="prefix" default="" />
+  <xacro:arg name="prefix" default=""/>
   <xacro:include filename="$(find ur_moveit_config)/srdf/ur_macro.srdf.xacro"/>
+  <xacro:include filename="$(find ur_moveit_config)/srdf/robotiq_85_gripper.srdf.xacro"/>
   <xacro:ur_srdf name="$(arg name)" prefix="$(arg prefix)"/>
+  <disable_collisions link1="$(arg prefix)robotiq_85_base_link" link2="$(arg prefix)tool0" reason="Adjacent" />
+  <disable_collisions link1="$(arg prefix)robotiq_85_base_link" link2="$(arg prefix)wrist_3_link" reason="Never" />
 </robot>

File: ur_moveit_config/srdf/ur_macro.srdf.xacro (robot description, xacro)
@@ -14,5 +14,5 @@
       <chain base_link="${prefix}base_link" tip_link="${prefix}tool0" />
     </group>
-    <group name="${prefix}gripper">
+<!--    <group name="${prefix}gripper">
       <chain base_link="${prefix}robotiq_85_base_link" tip_link="${prefix}robotiq_85_left_knuckle_link" />
       <chain base_link="${prefix}robotiq_85_base_link" tip_link="${prefix}robotiq_85_right_finger_tip_link" />
@@ -24,4 +24,5 @@
       <joint name="${prefix}robotiq_85_right_knuckle_joint"/>
     </group>
+ -->
     <group name="${prefix}arm_gripper">
         <group name="${prefix}${name}_manipulator" />
@@ -30,10 +31,4 @@
     </group>
     <!--GROUP STATES - Purpose - Define a named state for a particular group, in terms of joint values. This is useful to define states like 'folded arms'-->
-     <group_state name="${prefix}open" group="${prefix}gripper">
-      <joint name="${prefix}robotiq_85_left_knuckle_joint" value="0.0" />
-    </group_state>
-    <group_state name="${prefix}close" group="${prefix}gripper">
-      <joint name="${prefix}robotiq_85_left_knuckle_joint" value="0.8" />
-    </group_state>
     <group_state name="${prefix}home" group="${prefix}${name}_manipulator">
       <joint name="${prefix}elbow_joint" value="0" />
@@ -114,23 +109,4 @@
     <disable_collisions link1="${prefix}wrist_1_link" link2="${prefix}wrist_3_link" reason="Never" />
     <disable_collisions link1="${prefix}wrist_2_link" link2="${prefix}wrist_3_link" reason="Adjacent" />
-    <disable_collisions link1="${prefix}robotiq_85_base_link" link2="${prefix}tool0" reason="Adjacent" />
-    <disable_collisions link1="${prefix}robotiq_85_base_link" link2="${prefix}wrist_3_link" reason="Never" />
-    <disable_collisions link1="${prefix}robotiq_85_base_link" link2="${prefix}robotiq_85_left_knuckle_link" reason="Adjacent" />
-    <disable_collisions link1="${prefix}robotiq_85_base_link" link2="${prefix}robotiq_85_right_knuckle_link" reason="Adjacent" />
-    <disable_collisions link1="${prefix}robotiq_85_base_link" link2="${prefix}robotiq_85_left_inner_knuckle_link" reason="Adjacent" />
-    <disable_collisions link1="${prefix}robotiq_85_base_link" link2="${prefix}robotiq_85_right_inner_knuckle_link" reason="Adjacent" />
-    <disable_collisions link1="${prefix}robotiq_85_left_knuckle_link" link2="${prefix}robotiq_85_left_inner_knuckle_link" reason="Never" />
-    <disable_collisions link1="${prefix}robotiq_85_left_knuckle_link" link2="${prefix}robotiq_85_left_finger_link" reason="Adjacent" />
-    <disable_collisions link1="${prefix}robotiq_85_left_knuckle_link" link2="${prefix}robotiq_85_left_finger_tip_link" reason="Adjacent" />
-    <disable_collisions link1="${prefix}robotiq_85_right_knuckle_link" link2="${prefix}robotiq_85_right_inner_knuckle_link" reason="Never" />
-    <disable_collisions link1="${prefix}robotiq_85_right_knuckle_link" link2="${prefix}robotiq_85_right_finger_link" reason="Adjacent" />
-    <disable_collisions link1="${prefix}robotiq_85_right_knuckle_link" link2="${prefix}robotiq_85_right_finger_tip_link" reason="Adjacent" />
-    <disable_collisions link1="${prefix}robotiq_85_left_inner_knuckle_link" link2="${prefix}robotiq_85_right_inner_knuckle_link" reason="Never" />
-    <disable_collisions link1="${prefix}robotiq_85_left_inner_knuckle_link" link2="${prefix}robotiq_85_left_finger_link" reason="Adjacent" />
-    <disable_collisions link1="${prefix}robotiq_85_left_inner_knuckle_link" link2="${prefix}robotiq_85_left_finger_tip_link" reason="Adjacent" />
-    <disable_collisions link1="${prefix}robotiq_85_right_inner_knuckle_link" link2="${prefix}robotiq_85_right_finger_link" reason="Adjacent" />
-    <disable_collisions link1="${prefix}robotiq_85_right_inner_knuckle_link" link2="${prefix}robotiq_85_right_finger_tip_link" reason="Adjacent" />
-    <disable_collisions link1="${prefix}robotiq_85_left_finger_link" link2="${prefix}robotiq_85_left_finger_tip_link" reason="Adjacent" />
-    <disable_collisions link1="${prefix}robotiq_85_right_finger_link" link2="${prefix}robotiq_85_right_finger_tip_link" reason="Adjacent" />
   </xacro:macro>
 </robot>

Commit message: added us_gripper flag

File: ur_moveit_config/srdf/ur.srdf.xacro (robot description, xacro)
@@ -5,8 +5,14 @@
   <!-- parameters -->
   <xacro:arg name="prefix" default=""/>
+  <!-- Flag to use the Gripper or just the UR5  -->
+  <xacro:arg name="use_gripper" default="true" />
   <xacro:include filename="$(find ur_moveit_config)/srdf/ur_macro.srdf.xacro"/>
+  <xacro:if value="$(arg use_gripper)">
   <xacro:include filename="$(find ur_moveit_config)/srdf/robotiq_85_gripper.srdf.xacro"/>
-  <xacro:ur_srdf name="$(arg name)" prefix="$(arg prefix)"/>
+  </xacro:if>
+  <xacro:ur_srdf name="$(arg name)" prefix="$(arg prefix)" use_gripper="$(arg use_gripper)"/>
+  <xacro:if value="$(arg use_gripper)">
   <disable_collisions link1="$(arg prefix)robotiq_85_base_link" link2="$(arg prefix)tool0" reason="Adjacent" />
   <disable_collisions link1="$(arg prefix)robotiq_85_base_link" link2="$(arg prefix)wrist_3_link" reason="Never" />
+  </xacro:if>
 </robot>

File: ur_moveit_config/srdf/ur_macro.srdf.xacro (robot description, xacro)
@@ -5,5 +5,5 @@
     A URDF file must exist for this robot as well, where the joints and the links that are referenced are defined
 -->
-  <xacro:macro name="ur_srdf" params="name prefix">
+  <xacro:macro name="ur_srdf" params="name prefix use_gripper">
     <!--GROUPS - Representation of a set of joints and links. This can be useful for specifying DOF to plan for, defining arms, end effectors, etc-->
     <!--LINKS - When a link is specified, the parent joint of that link (if it exists) is automatically included-->
