Commit message: updating code

File: ur_moveit_config/srdf/robotiq_85_gripper.srdf.xacro (robot description, xacro)
@@ -1,6 +1,6 @@
 <?xml version='1.0' encoding='utf-8'?>
 <robot xmlns:xacro="http://www.ros.org/wiki/xacro" name="robotiq_85_gripper">
-  <xacro:arg name="prefix" default="" />
+  <xacro:arg name="tf_prefix" default="" />
   <xacro:include filename="$(find ur_moveit_config)/srdf/robotiq_85_gripper_macro.srdf.xacro"/>
-  <xacro:robotiq_85_gripper_srdf prefix="$(arg prefix)"/>
+  <xacro:robotiq_85_gripper_srdf tf_prefix="$(arg tf_prefix)"/>
 </robot>

File: ur_moveit_config/srdf/robotiq_85_gripper_macro.srdf.xacro (robot description, xacro)
@@ -1,50 +1,50 @@
 <?xml version="1.0" ?>
 <robot xmlns:xacro="http://www.ros.org/wiki/xacro" name="robotiq_85_gripper">
-  <xacro:macro name="robotiq_85_gripper_srdf" params="prefix">
-    <group name="${prefix}gripper">
-      <chain base_link="${prefix}robotiq_85_base_link" tip_link="${prefix}robotiq_85_left_knuckle_link" />
-      <chain base_link="${prefix}robotiq_85_base_link" tip_link="${prefix}robotiq_85_right_finger_tip_link" />
-      <chain base_link="${prefix}robotiq_85_base_link" tip_link="${prefix}robotiq_85_left_finger_tip_link" />
-      <link name="${prefix}robotiq_85_base_link"/>
-      <link name="${prefix}robotiq_85_left_knuckle_link"/>
-      <link name="${prefix}robotiq_85_right_knuckle_link"/>
-      <joint name="${prefix}robotiq_85_left_knuckle_joint"/>
-      <joint name="${prefix}robotiq_85_right_knuckle_joint"/>
+  <xacro:macro name="robotiq_85_gripper_srdf" params="tf_prefix">
+    <group name="${tf_prefix}gripper">
+      <chain base_link="${tf_prefix}robotiq_85_base_link" tip_link="${tf_prefix}robotiq_85_left_knuckle_link" />
+      <chain base_link="${tf_prefix}robotiq_85_base_link" tip_link="${tf_prefix}robotiq_85_right_finger_tip_link" />
+      <chain base_link="${tf_prefix}robotiq_85_base_link" tip_link="${tf_prefix}robotiq_85_left_finger_tip_link" />
+      <link name="${tf_prefix}robotiq_85_base_link"/>
+      <link name="${tf_prefix}robotiq_85_left_knuckle_link"/>
+      <link name="${tf_prefix}robotiq_85_right_knuckle_link"/>
+      <joint name="${tf_prefix}robotiq_85_left_knuckle_joint"/>
+      <joint name="${tf_prefix}robotiq_85_right_knuckle_joint"/>
     </group>
-    <group_state name="${prefix}open" group="${prefix}gripper">
-      <joint name="${prefix}robotiq_85_left_knuckle_joint" value="0.0" />
+    <group_state name="${tf_prefix}open" group="${tf_prefix}gripper">
+      <joint name="${tf_prefix}robotiq_85_left_knuckle_joint" value="0.0" />
     </group_state>
-    <group_state name="${prefix}close" group="${prefix}gripper">
-      <joint name="${prefix}robotiq_85_left_knuckle_joint" value="0.78" />
+    <group_state name="${tf_prefix}close" group="${tf_prefix}gripper">
+      <joint name="${tf_prefix}robotiq_85_left_knuckle_joint" value="0.78" />
     </group_state>
-    <group_state name="${prefix}almost_close" group="${prefix}gripper">
-      <joint name="${prefix}robotiq_85_left_knuckle_joint" value="0.7" />
+    <group_state name="${tf_prefix}almost_close" group="${tf_prefix}gripper">
+      <joint name="${tf_prefix}robotiq_85_left_knuckle_joint" value="0.7" />
     </group_state>
-    <group_state name="${prefix}half_open" group="${prefix}gripper">
-      <joint name="${prefix}robotiq_85_left_knuckle_joint" value="0.4" />
+    <group_state name="${tf_prefix}half_open" group="${tf_prefix}gripper">
+      <joint name="${tf_prefix}robotiq_85_left_knuckle_joint" value="0.4" />
     </group_state>
-    <group_state name="${prefix}open_5cm" group="${prefix}gripper">
-      <joint name="${prefix}robotiq_85_left_knuckle_joint" value="0.35" />
+    <group_state name="${tf_prefix}open_5cm" group="${tf_prefix}gripper">
+      <joint name="${tf_prefix}robotiq_85_left_knuckle_joint" value="0.35" />
     </group_state>
-    <group_state name="${prefix}push_5cm" group="${prefix}gripper">
-      <joint name="${prefix}robotiq_85_left_knuckle_joint" value="0.5" />
+    <group_state name="${tf_prefix}push_5cm" group="${tf_prefix}gripper">
+      <joint name="${tf_prefix}robotiq_85_left_knuckle_joint" value="0.5" />
     </group_state>
-    <disable_collisions link1="${prefix}robotiq_85_base_link" link2="${prefix}robotiq_85_left_knuckle_link" reason="Adjacent" />
-    <disable_collisions link1="${prefix}robotiq_85_base_link" link2="${prefix}robotiq_85_right_knuckle_link" reason="Adjacent" />
-    <disable_collisions link1="${prefix}robotiq_85_base_link" link2="${prefix}robotiq_85_left_inner_knuckle_link" reason="Adjacent" />
-    <disable_collisions link1="${prefix}robotiq_85_base_link" link2="${prefix}robotiq_85_right_inner_knuckle_link" reason="Adjacent" />
-    <disable_collisions link1="${prefix}robotiq_85_left_knuckle_link" link2="${prefix}robotiq_85_left_inner_knuckle_link" reason="Never" />
-    <disable_collisions link1="${prefix}robotiq_85_left_knuckle_link" link2="${prefix}robotiq_85_left_finger_link" reason="Adjacent" />
-    <disable_collisions link1="${prefix}robotiq_85_left_knuckle_link" link2="${prefix}robotiq_85_left_finger_tip_link" reason="Adjacent" />
-    <disable_collisions link1="${prefix}robotiq_85_right_knuckle_link" link2="${prefix}robotiq_85_right_inner_knuckle_link" reason="Never" />
-    <disable_collisions link1="${prefix}robotiq_85_right_knuckle_link" link2="${prefix}robotiq_85_right_finger_link" reason="Adjacent" />
-    <disable_collisions link1="${prefix}robotiq_85_right_knuckle_link" link2="${prefix}robotiq_85_right_finger_tip_link" reason="Adjacent" />
-    <disable_collisions link1="${prefix}robotiq_85_left_inner_knuckle_link" link2="${prefix}robotiq_85_right_inner_knuckle_link" reason="Never" />
-    <disable_collisions link1="${prefix}robotiq_85_left_inner_knuckle_link" link2="${prefix}robotiq_85_left_finger_link" reason="Adjacent" />
-    <disable_collisions link1="${prefix}robotiq_85_left_inner_knuckle_link" link2="${prefix}robotiq_85_left_finger_tip_link" reason="Adjacent" />
-    <disable_collisions link1="${prefix}robotiq_85_right_inner_knuckle_link" link2="${prefix}robotiq_85_right_finger_link" reason="Adjacent" />
-    <disable_collisions link1="${prefix}robotiq_85_right_inner_knuckle_link" link2="${prefix}robotiq_85_right_finger_tip_link" reason="Adjacent" />
-    <disable_collisions link1="${prefix}robotiq_85_left_finger_link" link2="${prefix}robotiq_85_left_finger_tip_link" reason="Adjacent" />
-    <disable_collisions link1="${prefix}robotiq_85_right_finger_link" link2="${prefix}robotiq_85_right_finger_tip_link" reason="Adjacent" />
+    <disable_collisions link1="${tf_prefix}robotiq_85_base_link" link2="${tf_prefix}robotiq_85_left_knuckle_link" reason="Adjacent" />
+    <disable_collisions link1="${tf_prefix}robotiq_85_base_link" link2="${tf_prefix}robotiq_85_right_knuckle_link" reason="Adjacent" />
+    <disable_collisions link1="${tf_prefix}robotiq_85_base_link" link2="${tf_prefix}robotiq_85_left_inner_knuckle_link" reason="Adjacent" />
+    <disable_collisions link1="${tf_prefix}robotiq_85_base_link" link2="${tf_prefix}robotiq_85_right_inner_knuckle_link" reason="Adjacent" />
+    <disable_collisions link1="${tf_prefix}robotiq_85_left_knuckle_link" link2="${tf_prefix}robotiq_85_left_inner_knuckle_link" reason="Never" />
+    <disable_collisions link1="${tf_prefix}robotiq_85_left_knuckle_link" link2="${tf_prefix}robotiq_85_left_finger_link" reason="Adjacent" />
+    <disable_collisions link1="${tf_prefix}robotiq_85_left_knuckle_link" link2="${tf_prefix}robotiq_85_left_finger_tip_link" reason="Adjacent" />
+    <disable_collisions link1="${tf_prefix}robotiq_85_right_knuckle_link" link2="${tf_prefix}robotiq_85_right_inner_knuckle_link" reason="Never" />
+    <disable_collisions link1="${tf_prefix}robotiq_85_right_knuckle_link" link2="${tf_prefix}robotiq_85_right_finger_link" reason="Adjacent" />
+    <disable_collisions link1="${tf_prefix}robotiq_85_right_knuckle_link" link2="${tf_prefix}robotiq_85_right_finger_tip_link" reason="Adjacent" />
+    <disable_collisions link1="${tf_prefix}robotiq_85_left_inner_knuckle_link" link2="${tf_prefix}robotiq_85_right_inner_knuckle_link" reason="Never" />
+    <disable_collisions link1="${tf_prefix}robotiq_85_left_inner_knuckle_link" link2="${tf_prefix}robotiq_85_left_finger_link" reason="Adjacent" />
+    <disable_collisions link1="${tf_prefix}robotiq_85_left_inner_knuckle_link" link2="${tf_prefix}robotiq_85_left_finger_tip_link" reason="Adjacent" />
+    <disable_collisions link1="${tf_prefix}robotiq_85_right_inner_knuckle_link" link2="${tf_prefix}robotiq_85_right_finger_link" reason="Adjacent" />
+    <disable_collisions link1="${tf_prefix}robotiq_85_right_inner_knuckle_link" link2="${tf_prefix}robotiq_85_right_finger_tip_link" reason="Adjacent" />
+    <disable_collisions link1="${tf_prefix}robotiq_85_left_finger_link" link2="${tf_prefix}robotiq_85_left_finger_tip_link" reason="Adjacent" />
+    <disable_collisions link1="${tf_prefix}robotiq_85_right_finger_link" link2="${tf_prefix}robotiq_85_right_finger_tip_link" reason="Adjacent" />
   </xacro:macro>
 </robot>

File: ur_moveit_config/srdf/ur.srdf.xacro (robot description, xacro)
@@ -4,5 +4,5 @@
   <xacro:arg name="name" default="ur"/>
   <!-- parameters -->
-  <xacro:arg name="prefix" default=""/>
+  <xacro:arg name="tf_prefix" default=""/>
   <!-- Flag to use the Gripper or just the UR5  -->
   <xacro:arg name="use_gripper" default="true" />
@@ -11,8 +11,8 @@
   <xacro:include filename="$(find ur_moveit_config)/srdf/robotiq_85_gripper.srdf.xacro"/>
   </xacro:if>
-  <xacro:ur_srdf name="$(arg name)" prefix="$(arg prefix)" use_gripper="$(arg use_gripper)"/>
+  <xacro:ur_srdf name="$(arg name)" tf_prefix="$(arg tf_prefix)" use_gripper="$(arg use_gripper)"/>
   <xacro:if value="$(arg use_gripper)">
-  <disable_collisions link1="$(arg prefix)robotiq_85_base_link" link2="$(arg prefix)tool0" reason="Adjacent" />
-  <disable_collisions link1="$(arg prefix)robotiq_85_base_link" link2="$(arg prefix)wrist_3_link" reason="Never" />
+  <disable_collisions link1="$(arg tf_prefix)robotiq_85_base_link" link2="$(arg tf_prefix)tool0" reason="Adjacent" />
+  <disable_collisions link1="$(arg tf_prefix)robotiq_85_base_link" link2="$(arg tf_prefix)wrist_3_link" reason="Never" />
   </xacro:if>
 </robot>
