Commit message: updating code

File: ur_moveit_config/srdf/ur_macro.srdf.xacro (robot description, xacro)
@@ -5,5 +5,5 @@
     A URDF file must exist for this robot as well, where the joints and the links that are referenced are defined
 -->
-  <xacro:macro name="ur_srdf" params="name prefix use_gripper">
+  <xacro:macro name="ur_srdf" params="name tf_prefix use_gripper">
     <!--GROUPS - Representation of a set of joints and links. This can be useful for specifying DOF to plan for, defining arms, end effectors, etc-->
     <!--LINKS - When a link is specified, the parent joint of that link (if it exists) is automatically included-->
@@ -11,102 +11,103 @@
     <!--CHAINS - When a chain is specified, all the links along the chain (including endpoints) are included in the group. Additionally, all the joints that are parents to included links are also included. This means that joints along the chain and the parent joint of the base link are included in the group-->
     <!--SUBGROUPS - Groups can also be formed by referencing to already defined group names-->
-    <group name="${prefix}${name}_manipulator">
-      <chain base_link="${prefix}base_link" tip_link="${prefix}tool0" />
+    <group name="${tf_prefix}${name}_manipulator">
+      <chain base_link="${tf_prefix}base_link" tip_link="${tf_prefix}tool0" />
     </group>
-<!--    <group name="${prefix}gripper">
-      <chain base_link="${prefix}robotiq_85_base_link" tip_link="${prefix}robotiq_85_left_knuckle_link" />
-      <chain base_link="${prefix}robotiq_85_base_link" tip_link="${prefix}robotiq_85_right_finger_tip_link" />
-      <chain base_link="${prefix}robotiq_85_base_link" tip_link="${prefix}robotiq_85_left_finger_tip_link" />
-      <link name="${prefix}robotiq_85_base_link"/>
-      <link name="${prefix}robotiq_85_left_knuckle_link"/>
-      <link name="${prefix}robotiq_85_right_knuckle_link"/>
-      <joint name="${prefix}robotiq_85_left_knuckle_joint"/>
-      <joint name="${prefix}robotiq_85_right_knuckle_joint"/>
+<!--    <group name="${tf_prefix}gripper">
+      <chain base_link="${tf_prefix}robotiq_85_base_link" tip_link="${tf_prefix}robotiq_85_left_knuckle_link" />
+      <chain base_link="${tf_prefix}robotiq_85_base_link" tip_link="${tf_prefix}robotiq_85_right_finger_tip_link" />
+      <chain base_link="${tf_prefix}robotiq_85_base_link" tip_link="${tf_prefix}robotiq_85_left_finger_tip_link" />
+      <link name="${tf_prefix}robotiq_85_base_link"/>
+      <link name="${tf_prefix}robotiq_85_left_knuckle_link"/>
+      <link name="${tf_prefix}robotiq_85_right_knuckle_link"/>
+      <joint name="${tf_prefix}robotiq_85_left_knuckle_joint"/>
+      <joint name="${tf_prefix}robotiq_85_right_knuckle_joint"/>
     </group>
  -->
-    <group name="${prefix}arm_gripper">
-        <group name="${prefix}${name}_manipulator" />
-        <joint name="${prefix}gripper_grasp_point_joint"/>
-        <link name="${prefix}gripper_grasp_point"/>
+    <group name="${tf_prefix}arm_gripper">
+        <group name="${tf_prefix}${name}_manipulator" />
+        <joint name="${tf_prefix}gripper_grasp_point_joint"/>
+        <link name="${tf_prefix}gripper_grasp_point"/>
     </group>
     <!--GROUP STATES - Purpose - Define a named state for a particular group, in terms of joint values. This is useful to define states like 'folded arms'-->
-    <group_state name="${prefix}home" group="${prefix}${name}_manipulator">
-      <joint name="${prefix}elbow_joint" value="0" />
-      <joint name="${prefix}shoulder_lift_joint" value="-1.5707" />
-      <joint name="${prefix}shoulder_pan_joint" value="0" />
-      <joint name="${prefix}wrist_1_joint" value="0" />
-      <joint name="${prefix}wrist_2_joint" value="0" />
-      <joint name="${prefix}wrist_3_joint" value="0" />
+    <group_state name="${tf_prefix}home" group="${tf_prefix}${name}_manipulator">
+      <joint name="${tf_prefix}elbow_joint" value="0" />
+      <joint name="${tf_prefix}shoulder_lift_joint" value="-1.5707" />
+      <joint name="${tf_prefix}shoulder_pan_joint" value="0" />
+      <joint name="${tf_prefix}wrist_1_joint" value="0" />
+      <joint name="${tf_prefix}wrist_2_joint" value="0" />
+      <joint name="${tf_prefix}wrist_3_joint" value="0" />
     </group_state>
-    <group_state name="${prefix}up" group="${prefix}${name}_manipulator">
-      <joint name="${prefix}elbow_joint" value="0" />
-      <joint name="${prefix}shoulder_lift_joint" value="-1.5707" />
-      <joint name="${prefix}shoulder_pan_joint" value="0" />
-      <joint name="${prefix}wrist_1_joint" value="-1.5707" />
-      <joint name="${prefix}wrist_2_joint" value="0" />
-      <joint name="${prefix}wrist_3_joint" value="0" />
+    <group_state name="${tf_prefix}up" group="${tf_prefix}${name}_manipulator">
+      <joint name="${tf_prefix}elbow_joint" value="0" />
+      <joint name="${tf_prefix}shoulder_lift_joint" value="-1.5707" />
+      <joint name="${tf_prefix}shoulder_pan_joint" value="0" />
+      <joint name="${tf_prefix}wrist_1_joint" value="-1.5707" />
+      <joint name="${tf_prefix}wrist_2_joint" value="0" />
+      <joint name="${tf_prefix}wrist_3_joint" value="0" />
     </group_state>
-    <group_state name="${prefix}test_configuration" group="${prefix}${name}_manipulator">
-      <joint name="${prefix}elbow_joint" value="1.4" />
-      <joint name="${prefix}shoulder_lift_joint" value="-1.62" />
-      <joint name="${prefix}shoulder_pan_joint" value="1.54" />
-      <joint name="${prefix}wrist_1_joint" value="-1.2" />
-      <joint name="${prefix}wrist_2_joint" value="-1.6" />
-      <joint name="${prefix}wrist_3_joint" value="-0.11" />
+    <group_state name="${tf_prefix}test_configuration" group="${tf_prefix}${name}_manipulator">
+      <joint name="${tf_prefix}elbow_joint" value="1.4" />
+      <joint name="${tf_prefix}shoulder_lift_joint" value="-1.62" />
+      <joint name="${tf_prefix}shoulder_pan_joint" value="1.54" />
+      <joint name="${tf_prefix}wrist_1_joint" value="-1.2" />
+      <joint name="${tf_prefix}wrist_2_joint" value="-1.6" />
+      <joint name="${tf_prefix}wrist_3_joint" value="-0.11" />
     </group_state>
-    <group_state name="${prefix}test_configuration" group="${prefix}arm_gripper">
-      <joint name="${prefix}elbow_joint" value="1.4" />
-      <joint name="${prefix}shoulder_lift_joint" value="-1.62" />
-      <joint name="${prefix}shoulder_pan_joint" value="1.54" />
-      <joint name="${prefix}wrist_1_joint" value="-1.2" />
-      <joint name="${prefix}wrist_2_joint" value="-1.6" />
-      <joint name="${prefix}wrist_3_joint" value="-0.0" />
+    <group_state name="${tf_prefix}test_configuration" group="${tf_prefix}arm_gripper">
+      <joint name="${tf_prefix}elbow_joint" value="1.4" />
+      <joint name="${tf_prefix}shoulder_lift_joint" value="-1.62" />
+      <joint name="${tf_prefix}shoulder_pan_joint" value="1.54" />
+      <joint name="${tf_prefix}wrist_1_joint" value="-1.2" />
+      <joint name="${tf_prefix}wrist_2_joint" value="-1.6" />
+      <joint name="${tf_prefix}wrist_3_joint" value="-0.0" />
     </group_state>
-    <group_state name="${prefix}pre_picking" group="${prefix}arm_gripper">
-      <joint name="${prefix}elbow_joint" value="1.4" />
-      <joint name="${prefix}shoulder_lift_joint" value="-1.62" />
-      <joint name="${prefix}shoulder_pan_joint" value="1.54" />
-      <joint name="${prefix}wrist_1_joint" value="-1.35" />
-      <joint name="${prefix}wrist_2_joint" value="-1.6" />
-      <joint name="${prefix}wrist_3_joint" value="-0.0" />
+    <group_state name="${tf_prefix}pre_picking" group="${tf_prefix}arm_gripper">
+      <joint name="${tf_prefix}elbow_joint" value="1.4" />
+      <joint name="${tf_prefix}shoulder_lift_joint" value="-1.62" />
+      <joint name="${tf_prefix}shoulder_pan_joint" value="1.54" />
+      <joint name="${tf_prefix}wrist_1_joint" value="-1.35" />
+      <joint name="${tf_prefix}wrist_2_joint" value="-1.6" />
+      <joint name="${tf_prefix}wrist_3_joint" value="-0.0" />
     </group_state>
-    <group_state name="${prefix}picking" group="${prefix}arm_gripper">
-      <joint name="${prefix}elbow_joint" value="1.605" />
-      <joint name="${prefix}shoulder_lift_joint" value="-1.64" />
-      <joint name="${prefix}shoulder_pan_joint" value="1.54" />
-      <joint name="${prefix}wrist_1_joint" value="-1.57" />
-      <joint name="${prefix}wrist_2_joint" value="-1.605" />
-      <joint name="${prefix}wrist_3_joint" value="-0.0" />
+    <group_state name="${tf_prefix}picking" group="${tf_prefix}arm_gripper">
+      <joint name="${tf_prefix}elbow_joint" value="1.605" />
+      <joint name="${tf_prefix}shoulder_lift_joint" value="-1.64" />
+      <joint name="${tf_prefix}shoulder_pan_joint" value="1.54" />
+      <joint name="${tf_prefix}wrist_1_joint" value="-1.57" />
+      <joint name="${tf_prefix}wrist_2_joint" value="-1.605" />
+      <joint name="${tf_prefix}wrist_3_joint" value="-0.0" />
     </group_state>
-    <group_state name="${prefix}pre_drop" group="${prefix}arm_gripper">
-      <joint name="${prefix}elbow_joint" value="1.37" />
-      <joint name="${prefix}shoulder_lift_joint" value="-1.59" />
-      <joint name="${prefix}shoulder_pan_joint" value="1.81" />
-      <joint name="${prefix}wrist_1_joint" value="-1.36" />
-      <joint name="${prefix}wrist_2_joint" value="-1.61" />
-      <joint name="${prefix}wrist_3_joint" value="0.26" />
+    <group_state name="${tf_prefix}pre_drop" group="${tf_prefix}arm_gripper">
+      <joint name="${tf_prefix}elbow_joint" value="1.37" />
+      <joint name="${tf_prefix}shoulder_lift_joint" value="-1.59" />
+      <joint name="${tf_prefix}shoulder_pan_joint" value="1.81" />
+      <joint name="${tf_prefix}wrist_1_joint" value="-1.36" />
+      <joint name="${tf_prefix}wrist_2_joint" value="-1.61" />
+      <joint name="${tf_prefix}wrist_3_joint" value="0.26" />
     </group_state>
-    <group_state name="${prefix}drop_off" group="${prefix}arm_gripper">
-      <joint name="${prefix}elbow_joint" value="1.57" />
-      <joint name="${prefix}shoulder_lift_joint" value="-1.61" />
-      <joint name="${prefix}shoulder_pan_joint" value="1.80" />
-      <joint name="${prefix}wrist_1_joint" value="-1.54" />
-      <joint name="${prefix}wrist_2_joint" value="-1.61" />
-      <joint name="${prefix}wrist_3_joint" value="0.26" />
+    <group_state name="${tf_prefix}drop_off" group="${tf_prefix}arm_gripper">
+      <joint name="${tf_prefix}elbow_joint" value="1.57" />
+      <joint name="${tf_prefix}shoulder_lift_joint" value="-1.61" />
+      <joint name="${tf_prefix}shoulder_pan_joint" value="1.80" />
+      <joint name="${tf_prefix}wrist_1_joint" value="-1.54" />
+      <joint name="${tf_prefix}wrist_2_joint" value="-1.61" />
+      <joint name="${tf_prefix}wrist_3_joint" value="0.26" />
     </group_state>
     <!--END EFFECTOR - Purpose - Represent information about an end effector.-->
     <!--VIRTUAL JOINT - Purpose - this element defines a virtual joint between a robot link and an external frame of reference (considered fixed with respect to the robot)-->
     <!--DISABLE COLLISIONS - By default it is assumed that any link of the robot could potentially come into collision with any other link in the robot. This tag disables collision checking between a specified pair of links. -->
-    <disable_collisions link1="${prefix}base_link" link2="${prefix}base_link_inertia" reason="Adjacent" />
-    <disable_collisions link1="${prefix}base_link_inertia" link2="${prefix}shoulder_link" reason="Adjacent" />
-    <disable_collisions link1="${prefix}tool0" link2="${prefix}wrist_1_link" reason="Never" />
-    <disable_collisions link1="${prefix}tool0" link2="${prefix}wrist_2_link" reason="Never" />
-    <disable_collisions link1="${prefix}tool0" link2="${prefix}wrist_3_link" reason="Adjacent" />
-    <disable_collisions link1="${prefix}forearm_link" link2="${prefix}upper_arm_link" reason="Adjacent" />
-    <disable_collisions link1="${prefix}forearm_link" link2="${prefix}wrist_1_link" reason="Adjacent" />
-    <disable_collisions link1="${prefix}shoulder_link" link2="${prefix}upper_arm_link" reason="Adjacent" />
-    <disable_collisions link1="${prefix}wrist_1_link" link2="${prefix}wrist_2_link" reason="Adjacent" />
-    <disable_collisions link1="${prefix}wrist_1_link" link2="${prefix}wrist_3_link" reason="Never" />
-    <disable_collisions link1="${prefix}wrist_2_link" link2="${prefix}wrist_3_link" reason="Adjacent" />
+    <disable_collisions link1="${tf_prefix}base_link" link2="${tf_prefix}base_link_inertia" reason="Adjacent" />
+    <disable_collisions link1="${tf_prefix}base_link_inertia" link2="${tf_prefix}shoulder_link" reason="Adjacent" />
+    <disable_collisions link1="${tf_prefix}base_link" link2="${tf_prefix}base" reason="Adjacent" />
+    <disable_collisions link1="${tf_prefix}tool0" link2="${tf_prefix}wrist_1_link" reason="Never" />
+    <disable_collisions link1="${tf_prefix}tool0" link2="${tf_prefix}wrist_2_link" reason="Never" />
+    <disable_collisions link1="${tf_prefix}tool0" link2="${tf_prefix}wrist_3_link" reason="Adjacent" />
+    <disable_collisions link1="${tf_prefix}forearm_link" link2="${tf_prefix}upper_arm_link" reason="Adjacent" />
+    <disable_collisions link1="${tf_prefix}forearm_link" link2="${tf_prefix}wrist_1_link" reason="Adjacent" />
+    <disable_collisions link1="${tf_prefix}shoulder_link" link2="${tf_prefix}upper_arm_link" reason="Adjacent" />
+    <disable_collisions link1="${tf_prefix}wrist_1_link" link2="${tf_prefix}wrist_2_link" reason="Adjacent" />
+    <disable_collisions link1="${tf_prefix}wrist_1_link" link2="${tf_prefix}wrist_3_link" reason="Never" />
+    <disable_collisions link1="${tf_prefix}wrist_2_link" link2="${tf_prefix}wrist_3_link" reason="Adjacent" />
   </xacro:macro>
 </robot>
